Commit message: cosmos3 urdf

File: cosmos3_robot/cosmos/robot_model/urdf/left_arm_with_wrist_camera.urdf (robot description, URDF)
Before this commit: robot left_ar5_with_wrist_camera, 34 links, 33 joints
Links:
- added link AR5-5_07R_base; collision mesh filename=package://robot_model/meshes/AR5_P_R/AR5-5_07R_base.stl scale=0.001 0.001 0.001; visual mesh filename=package://robot_model/meshes/AR5_P_R/AR5-5_07R_base.stl scale=0.001 0.001 0.001
- added link AR5-5_07R_link1, mass 2.66; collision mesh filename=package://robot_model/meshes/AR5_P_R/AR5-5_07R_link1.stl scale=0.001 0.001 0.001; visual mesh filename=package://robot_model/meshes/AR5_P_R/AR5-5_07R_link1.stl scale=0.001 0.001 0.001
- added link AR5-5_07R_link2, mass 2.3; collision mesh filename=package://robot_model/meshes/AR5_P_R/AR5-5_07R_link2.stl scale=0.001 0.001 0.001; visual mesh filename=package://robot_model/meshes/AR5_P_R/AR5-5_07R_link2.stl scale=0.001 0.001 0.001
- added link AR5-5_07R_link3, mass 1.8; collision mesh filename=package://robot_model/meshes/AR5_P_R/AR5-5_07R_link3.stl scale=0.001 0.001 0.001; visual mesh filename=package://robot_model/meshes/AR5_P_R/AR5-5_07R_link3.stl scale=0.001 0.001 0.001
- added link AR5-5_07R_link4, mass 1.13; collision mesh filename=package://robot_model/meshes/AR5_P_R/AR5-5_07R_link4.stl scale=0.001 0.001 0.001; visual mesh filename=package://robot_model/meshes/AR5_P_R/AR5-5_07R_link4.stl scale=.001 0.001 0.001
- added link AR5-5_07R_link5, mass 1.19; collision mesh filename=package://robot_model/meshes/AR5_P_R/AR5-5_07R_link5.stl scale=0.001 0.001 0.001; visual mesh filename=package://robot_model/meshes/AR5_P_R/AR5-5_07R_link5.stl scale=0.001 0.001 0.001
- added link AR5-5_07R_link6, mass 0.82; collision mesh filename=package://robot_model/meshes/AR5_P_R/AR5-5_07R_link6.stl scale=0.001 0.001 0.001; visual mesh filename=package://robot_model/meshes/AR5_P_R/AR5-5_07R_link6.stl scale=0.001 0.001 0.001
- added link AR5-5_07R_link7, mass 0.32; collision mesh filename=package://robot_model/meshes/AR5_P_R/AR5-5_07R_link7.stl scale=0.001 0.001 0.001; visual mesh filename=package://robot_model/meshes/AR5_P_R/AR5-5_07R_link7.stl scale=0.001 0.001 0.001
- added link AR5-5_07R_tcp, mass 0.0
- added link rh6_right_base_link, mass 0.211569079117232; collision mesh filename=package://robot_model/meshes/rh6_ctrl/base_linky.STL; visual mesh filename=package://robot_model/meshes/rh6_ctrl/base_linky.STL
- added link rh6_right_fz11_Link, mass 0.0122865280263998; collision mesh filename=package://robot_model/meshes/rh6_ctrl/fy11_Link.STL; visual mesh filename=package://robot_model/meshes/rh6_ctrl/fy11_Link.STL
- added link rh6_right_fz12_Link, mass 0.0125497959072737; collision mesh filename=package://robot_model/meshes/rh6_ctrl/fy12_Link.STL; visual mesh filename=package://robot_model/meshes/rh6_ctrl/fy12_Link.STL
- added link rh6_right_fz13_Link, mass 0.00766845638651249; collision mesh filename=package://robot_model/meshes/rh6_ctrl/fy13_Link.STL; visual mesh filename=package://robot_model/meshes/rh6_ctrl/fy13_Link.STL
- added link rh6_right_fz14_Link, mass 0.00378673281389124; collision mesh filename=package://robot_model/meshes/rh6_ctrl/fy14_Link.STL; visual mesh filename=package://robot_model/meshes/rh6_ctrl/fy14_Link.STL
- added link rh6_right_fz21_Link, mass 0.0100639225371382; collision mesh filename=package://robot_model/meshes/rh6_ctrl/fy21_Link.STL; visual mesh filename=package://robot_model/meshes/rh6_ctrl/fy21_Link.STL
- added link rh6_right_fz22_Link, mass 0.00358605495739092; collision mesh filename=package://robot_model/meshes/rh6_ctrl/fy22_Link.STL; visual mesh filename=package://robot_model/meshes/rh6_ctrl/fy22_Link.STL
- added link rh6_right_fz23_Link, mass 0.00260327905787072; collision mesh filename=package://robot_model/meshes/rh6_ctrl/fy23_Link.STL; visual mesh filename=package://robot_model/meshes/rh6_ctrl/fy23_Link.STL
- added link rh6_right_fz31_Link, mass 0.00829865569529675; collision mesh filename=package://robot_model/meshes/rh6_ctrl/fy31_Link.STL; visual mesh filename=package://robot_model/meshes/rh6_ctrl/fy31_Link.STL
- added link rh6_right_fz32_Link, mass 0.00358603535605245; collision mesh filename=package://robot_model/meshes/rh6_ctrl/fy32_Link.STL; visual mesh filename=package://robot_model/meshes/rh6_ctrl/fy32_Link.STL
- added link rh6_right_fz33_Link, mass 0.00260328811165374; collision mesh filename=package://robot_model/meshes/rh6_ctrl/fy33_Link.STL; visual mesh filename=package://robot_model/meshes/rh6_ctrl/fy33_Link.STL
- added link rh6_right_fz41_Link, mass 0.0100639366001575; collision mesh filename=package://robot_model/meshes/rh6_ctrl/fy41_Link.STL; visual mesh filename=package://robot_model/meshes/rh6_ctrl/fy41_Link.STL
- added link rh6_right_fz42_Link, mass 0.00358590544643104; collision mesh filename=package://robot_model/meshes/rh6_ctrl/fy42_Link.STL; visual mesh filename=package://robot_model/meshes/rh6_ctrl/fy42_Link.STL
- added link rh6_right_fz43_Link, mass 0.00260331123444047; collision mesh filename=package://robot_model/meshes/rh6_ctrl/fy43_Link.STL; visual mesh filename=package://robot_model/meshes/rh6_ctrl/fy43_Link.STL
- added link rh6_right_fz51_Link, mass 0.00870573306563604; collision mesh filename=package://robot_model/meshes/rh6_ctrl/fy51_Link.STL; visual mesh filename=package://robot_model/meshes/rh6_ctrl/fy51_Link.STL
- added link rh6_right_fz52_Link, mass 0.00358587967262367; collision mesh filename=package://robot_model/meshes/rh6_ctrl/fy52_Link.STL; visual mesh filename=package://robot_model/meshes/rh6_ctrl/fy52_Link.STL
- added link rh6_right_fz53_Link, mass 0.00260328769879583; collision mesh filename=package://robot_model/meshes/rh6_ctrl/fy53_Link.STL; visual mesh filename=package://robot_model/meshes/rh6_ctrl/fy53_Link.STL
- added link rh6_right_grasp_center; visual sphere radius=0.002
- added link right_wrist_camera_color_frame; visual sphere radius=0.008
- added link right_wrist_camera_link; visual mesh filename=package://robot_model/meshes/others_stl/Camera_435.stl scale=0.001 0.001 0.001
Joints:
- added joint AR5-5_07R_joint_1: type revolute, parent AR5-5_07R_base, child AR5-5_07R_link1, origin xyz=0.0 0.0 0.0 rpy=0 0 0, axis 0 0 1, limit lower=-3.1067 upper=3.1067 effort=108 velocity=3.490658503988659
- added joint AR5-5_07R_joint_2: type revolute, parent AR5-5_07R_link1, child AR5-5_07R_link2, origin xyz=0.0 0.0 0.1745 rpy=0 0 0, axis 0 1 0, limit lower=-2.0944 upper=2.0944 effort=108 velocity=3.490658503988659
- added joint AR5-5_07R_joint_3: type revolute, parent AR5-5_07R_link2, child AR5-5_07R_link3, origin xyz=0.0 0.0 0.314 rpy=0 0 0, axis 0 0 1, limit lower=-3.1067 upper=3.1067 effort=66 velocity=4.71238898038469
- added joint AR5-5_07R_joint_4: type revolute, parent AR5-5_07R_link3, child AR5-5_07R_link4, origin xyz=0.0105 0.0 0.0 rpy=0 0 0, axis 0 1 0, limit lower=-1.0472 upper=2.5307 effort=66 velocity=5.235987755982989
- added joint AR5-5_07R_joint_5: type revolute, parent AR5-5_07R_link4, child AR5-5_07R_link5, origin xyz=-0.0105 0.0 0.26 rpy=0 0 0, axis 0 0 1, limit lower=-3.1067 upper=3.1067 effort=19 velocity=4.1887902047863905
- added joint AR5-5_07R_joint_6: type revolute, parent AR5-5_07R_link5, child AR5-5_07R_link6, origin xyz=0.0 0.0 0.0 rpy=0.0 0.0 0, axis 0 1 0, limit lower=-1.0472 upper=1.0472 effort=19 velocity=4.1887902047863905
- added joint AR5-5_07R_joint_7: type revolute, parent AR5-5_07R_link6, child AR5-5_07R_link7, origin xyz=0.0 0.0 0.0 rpy=0.0 0.0 0, axis 1 0 0, limit lower=-1.0472 upper=1.0472 effort=19 velocity=4.1887902047863905
- added joint AR5-5_07R_tcp_joint: type fixed, parent AR5-5_07R_link7, child AR5-5_07R_tcp, origin xyz=0.001802 -0.000099 0.097 rpy=0 0 0
- added joint rh6_right_fz11: type revolute, parent rh6_right_base_link, child rh6_right_fz11_Link, origin xyz=0.0135 0.022 0.0398 rpy=0 0 1.5708, axis 0 0 -1, limit lower=0 upper=2.356 effort=0 velocity=0
- added joint rh6_right_fz12: type revolute, parent rh6_right_fz11_Link, child rh6_right_fz12_Link, origin xyz=0.0105 0 0.0107 rpy=1.5708 0 0, axis 0 0 1, limit lower=0 upper=0.698 effort=0 velocity=0
- added joint rh6_right_fz13: type revolute, parent rh6_right_fz12_Link, child rh6_right_fz13_Link, origin xyz=0.040457 0.011223 0 rpy=0 0 0, axis 0 0 1, limit lower=0 upper=1.169 effort=0 velocity=0
- added joint rh6_right_fz14: type revolute, parent rh6_right_fz13_Link, child rh6_right_fz14_Link, origin xyz=0.036284 0.0268 0 rpy=-0.36834 1.5708 0, axis 0 0 1, limit lower=0 upper=0 effort=0 velocity=0
- added joint rh6_right_fz21: type revolute, parent rh6_right_base_link, child rh6_right_fz21_Link, origin xyz=-0.0035 0.029833 0.11095 rpy=0 -1.4923 1.5708, axis 0 0 -1, limit lower=0 upper=1.518 effort=0 velocity=0
- added joint rh6_right_fz22: type revolute, parent rh6_right_fz21_Link, child rh6_right_fz22_Link, origin xyz=0.0419 0.001 0 rpy=0 0 0, axis 0 0 -1, limit lower=0 upper=1.623 effort=0 velocity=0
- added joint rh6_right_fz23: type revolute, parent rh6_right_fz22_Link, child rh6_right_fz23_Link, origin xyz=0.043692 -0.011217 0 rpy=-1.5708 1.5695 -1.5543, axis 0 0 -1, limit lower=0 upper=0 effort=0 velocity=0
- added joint rh6_right_fz31: type revolute, parent rh6_right_base_link, child rh6_right_fz31_Link, origin xyz=-0.0035 0.009945 0.112 rpy=0 -1.5446 1.5708, axis 0 0 -1, limit lower=0 upper=1.571 effort=0 velocity=0
- added joint rh6_right_fz32: type revolute, parent rh6_right_fz31_Link, child rh6_right_fz32_Link, origin xyz=0.0519 0.001 0 rpy=0 0 0, axis 0 0 -1, limit lower=0 upper=1.641 effort=0 velocity=0
- added joint rh6_right_fz33: type revolute, parent rh6_right_fz32_Link, child rh6_right_fz33_Link, origin xyz=0.043641 -0.01141 0 rpy=-1.5708 1.5705 -1.5587, axis 0 0 -1, limit lower=0 upper=0 effort=0 velocity=0
- added joint rh6_right_fz41: type revolute, parent rh6_right_base_link, child rh6_right_fz41_Link, origin xyz=-0.0035 -0.009945 0.11099 rpy=3.1416 -1.5446 -1.5708, axis 0 0 -1, limit lower=0 upper=1.571 effort=0 velocity=0
- added joint rh6_right_fz42: type revolute, parent rh6_right_fz41_Link, child rh6_right_fz42_Link, origin xyz=0.0419 0.001 0 rpy=0 0 0, axis 0 0 -1, limit lower=0 upper=1.658 effort=0 velocity=0
- added joint rh6_right_fz43: type revolute, parent rh6_right_fz42_Link, child rh6_right_fz43_Link, origin xyz=0.043692 -0.011217 0 rpy=1.5708 1.5704 1.5873, axis 0 0 -1, limit lower=0 upper=0 effort=0 velocity=0
- added joint rh6_right_fz51: type revolute, parent rh6_right_base_link, child rh6_right_fz51_Link, origin xyz=-0.0035 -0.029624 0.10795 rpy=3.1416 -1.4923 -1.5708, axis 0 0 -1, limit lower=0 upper=1.545 effort=0 velocity=0
- added joint rh6_right_fz52: type revolute, parent rh6_right_fz51_Link, child rh6_right_fz52_Link, origin xyz=0.0369 0.001 0 rpy=0 0 0, axis 0 0 -1, limit lower=0 upper=1.658 effort=0 velocity=0
- added joint rh6_right_fz53: type revolute, parent rh6_right_fz52_Link, child rh6_right_fz53_Link, origin xyz=0.043691 -0.011217 0 rpy=1.5708 1.5695 1.5873, axis 0 0 -1, limit lower=0 upper=0 effort=0 velocity=0
- added joint rh6_right_grasp_center_joint: type fixed, parent rh6_right_base_link, child rh6_right_grasp_center, origin xyz=0.02 0 0.1 rpy=0 0 0
- added joint right_fixed: type fixed, parent basement_base_link, child AR5-5_07R_base, origin xyz=0.10645 0 1.40 rpy=0 1.5707963267948966 0
- added joint right_rh6_mount_joint: type fixed, parent AR5-5_07R_tcp, child rh6_right_base_link, origin xyz=0 0 0.01025 rpy=0 0 0
- added joint right_wrist_camera_color_fixed: type fixed, parent right_wrist_camera_link, child right_wrist_camera_color_frame, origin xyz=0 0 0 rpy=0 0 0
- added joint right_wrist_camera_fixed: type fixed, parent AR5-5_07R_tcp, child right_wrist_camera_link, origin xyz=-0.1 0 0 rpy=0 -1.570796327 0

Commit message: Finished the  urdf for the test robot

File: cosmos3_robot/cosmos/robot_model/urdf/left_arm_with_wrist_camera.urdf (robot description, URDF)
Before this commit: robot left_ar5_with_wrist_camera, 63 links, 62 joints
Links:
- removed link rh6_right_fz11_Link
- removed link rh6_right_fz12_Link
- removed link rh6_right_fz13_Link
- removed link rh6_right_fz14_Link
- removed link rh6_right_fz21_Link
- removed link rh6_right_fz22_Link
- removed link rh6_right_fz23_Link
- removed link rh6_right_fz31_Link
- removed link rh6_right_fz32_Link
- removed link rh6_right_fz33_Link
- removed link rh6_right_fz41_Link
- removed link rh6_right_fz42_Link
- removed link rh6_right_fz43_Link
- removed link rh6_right_fz51_Link
- removed link rh6_right_fz52_Link
- removed link rh6_right_fz53_Link
- added link rh6_right_fy11_Link, mass 0.0122865280263998; collision mesh filename=package://robot_model/meshes/rh6_ctrl/fy11_Link.STL; visual mesh filename=package://robot_model/meshes/rh6_ctrl/fy11_Link.STL
- added link rh6_right_fy12_Link, mass 0.0125497959072737; collision mesh filename=package://robot_model/meshes/rh6_ctrl/fy12_Link.STL; visual mesh filename=package://robot_model/meshes/rh6_ctrl/fy12_Link.STL
- added link rh6_right_fy13_Link, mass 0.00766845638651249; collision mesh filename=package://robot_model/meshes/rh6_ctrl/fy13_Link.STL; visual mesh filename=package://robot_model/meshes/rh6_ctrl/fy13_Link.STL
- added link rh6_right_fy14_Link, mass 0.00378673281389124; collision mesh filename=package://robot_model/meshes/rh6_ctrl/fy14_Link.STL; visual mesh filename=package://robot_model/meshes/rh6_ctrl/fy14_Link.STL
- added link rh6_right_fy21_Link, mass 0.0100639225371382; collision mesh filename=package://robot_model/meshes/rh6_ctrl/fy21_Link.STL; visual mesh filename=package://robot_model/meshes/rh6_ctrl/fy21_Link.STL
- added link rh6_right_fy22_Link, mass 0.00358605495739092; collision mesh filename=package://robot_model/meshes/rh6_ctrl/fy22_Link.STL; visual mesh filename=package://robot_model/meshes/rh6_ctrl/fy22_Link.STL
- added link rh6_right_fy23_Link, mass 0.00260327905787072; collision mesh filename=package://robot_model/meshes/rh6_ctrl/fy23_Link.STL; visual mesh filename=package://robot_model/meshes/rh6_ctrl/fy23_Link.STL
- added link rh6_right_fy31_Link, mass 0.00829865569529675; collision mesh filename=package://robot_model/meshes/rh6_ctrl/fy31_Link.STL; visual mesh filename=package://robot_model/meshes/rh6_ctrl/fy31_Link.STL
- added link rh6_right_fy32_Link, mass 0.00358603535605245; collision mesh filename=package://robot_model/meshes/rh6_ctrl/fy32_Link.STL; visual mesh filename=package://robot_model/meshes/rh6_ctrl/fy32_Link.STL
- added link rh6_right_fy33_Link, mass 0.00260328811165374; collision mesh filename=package://robot_model/meshes/rh6_ctrl/fy33_Link.STL; visual mesh filename=package://robot_model/meshes/rh6_ctrl/fy33_Link.STL
- added link rh6_right_fy41_Link, mass 0.0100639366001575; collision mesh filename=package://robot_model/meshes/rh6_ctrl/fy41_Link.STL; visual mesh filename=package://robot_model/meshes/rh6_ctrl/fy41_Link.STL
- added link rh6_right_fy42_Link, mass 0.00358590544643104; collision mesh filename=package://robot_model/meshes/rh6_ctrl/fy42_Link.STL; visual mesh filename=package://robot_model/meshes/rh6_ctrl/fy42_Link.STL
- added link rh6_right_fy43_Link, mass 0.00260331123444047; collision mesh filename=package://robot_model/meshes/rh6_ctrl/fy43_Link.STL; visual mesh filename=package://robot_model/meshes/rh6_ctrl/fy43_Link.STL
- added link rh6_right_fy51_Link, mass 0.00870573306563604; collision mesh filename=package://robot_model/meshes/rh6_ctrl/fy51_Link.STL; visual mesh filename=package://robot_model/meshes/rh6_ctrl/fy51_Link.STL
- added link rh6_right_fy52_Link, mass 0.00358587967262367; collision mesh filename=package://robot_model/meshes/rh6_ctrl/fy52_Link.STL; visual mesh filename=package://robot_model/meshes/rh6_ctrl/fy52_Link.STL
- added link rh6_right_fy53_Link, mass 0.00260328769879583; collision mesh filename=package://robot_model/meshes/rh6_ctrl/fy53_Link.STL; visual mesh filename=package://robot_model/meshes/rh6_ctrl/fy53_Link.STL
- link camera_base_link: geometry collision mesh filename=package://robot_model/meshes/722胸向前海康工业摄像头架子.STL scale=0.001 0.001 0.001; visual mesh filename=package://robot_model/meshes/722胸向前海康工业摄像头架子.STL scale=0.001 0.001 0.001
- link camera_link: geometry collision mesh filename=package://robot_model/meshes/MV-CU013-A0GMGC.STL scale=0.001 0.001 0.001; visual mesh filename=package://robot_model/meshes/MV-CU013-A0GMGC.STL scale=0.001 0.001 0.001
- link left_wrist_camera_link: geometry collision box size=0.023 0.042 0.042; visual mesh filename=package://robot_model/meshes/others_stl/D405.stl scale=0.001 0.001 0.001
- link right_wrist_camera_link: geometry collision box size=0.023 0.042 0.042; visual mesh filename=package://robot_model/meshes/others_stl/D405.stl scale=0.001 0.001 0.001
Joints:
- removed joint rh6_right_fz11
- removed joint rh6_right_fz12
- removed joint rh6_right_fz13
- removed joint rh6_right_fz14
- removed joint rh6_right_fz21
- removed joint rh6_right_fz22
- removed joint rh6_right_fz23
- removed joint rh6_right_fz31
- removed joint rh6_right_fz32
- removed joint rh6_right_fz33
- removed joint rh6_right_fz41
- removed joint rh6_right_fz42
- removed joint rh6_right_fz43
- removed joint rh6_right_fz51
- removed joint rh6_right_fz52
- removed joint rh6_right_fz53
- added joint rh6_right_fy11: type revolute, parent rh6_right_base_link, child rh6_right_fy11_Link, origin xyz=0.0135 0.022 0.0398 rpy=0 0 1.5708, axis 0 0 -1, limit lower=0 upper=2.356 effort=0 velocity=0
- added joint rh6_right_fy12: type revolute, parent rh6_right_fy11_Link, child rh6_right_fy12_Link, origin xyz=0.0105 0 0.0107 rpy=1.5708 0 0, axis 0 0 1, limit lower=0 upper=0.698 effort=0 velocity=0
- added joint rh6_right_fy13: type revolute, parent rh6_right_fy12_Link, child rh6_right_fy13_Link, origin xyz=0.040457 0.011223 0 rpy=0 0 0, axis 0 0 1, limit lower=0 upper=1.169 effort=0 velocity=0
- added joint rh6_right_fy14: type revolute, parent rh6_right_fy13_Link, child rh6_right_fy14_Link, origin xyz=0.036284 0.0268 0 rpy=-0.36834 1.5708 0, axis 0 0 1, limit lower=0 upper=0 effort=0 velocity=0
- added joint rh6_right_fy21: type revolute, parent rh6_right_base_link, child rh6_right_fy21_Link, origin xyz=-0.0035 0.029833 0.11095 rpy=0 -1.4923 1.5708, axis 0 0 -1, limit lower=0 upper=1.518 effort=0 velocity=0
- added joint rh6_right_fy22: type revolute, parent rh6_right_fy21_Link, child rh6_right_fy22_Link, origin xyz=0.0419 0.001 0 rpy=0 0 0, axis 0 0 -1, limit lower=0 upper=1.623 effort=0 velocity=0
- added joint rh6_right_fy23: type revolute, parent rh6_right_fy22_Link, child rh6_right_fy23_Link, origin xyz=0.043692 -0.011217 0 rpy=-1.5708 1.5695 -1.5543, axis 0 0 -1, limit lower=0 upper=0 effort=0 velocity=0
- added joint rh6_right_fy31: type revolute, parent rh6_right_base_link, child rh6_right_fy31_Link, origin xyz=-0.0035 0.009945 0.112 rpy=0 -1.5446 1.5708, axis 0 0 -1, limit lower=0 upper=1.571 effort=0 velocity=0
- added joint rh6_right_fy32: type revolute, parent rh6_right_fy31_Link, child rh6_right_fy32_Link, origin xyz=0.0519 0.001 0 rpy=0 0 0, axis 0 0 -1, limit lower=0 upper=1.641 effort=0 velocity=0
- added joint rh6_right_fy33: type revolute, parent rh6_right_fy32_Link, child rh6_right_fy33_Link, origin xyz=0.043641 -0.01141 0 rpy=-1.5708 1.5705 -1.5587, axis 0 0 -1, limit lower=0 upper=0 effort=0 velocity=0
- added joint rh6_right_fy41: type revolute, parent rh6_right_base_link, child rh6_right_fy41_Link, origin xyz=-0.0035 -0.009945 0.11099 rpy=3.1416 -1.5446 -1.5708, axis 0 0 -1, limit lower=0 upper=1.571 effort=0 velocity=0
- added joint rh6_right_fy42: type revolute, parent rh6_right_fy41_Link, child rh6_right_fy42_Link, origin xyz=0.0419 0.001 0 rpy=0 0 0, axis 0 0 -1, limit lower=0 upper=1.658 effort=0 velocity=0
- added joint rh6_right_fy43: type revolute, parent rh6_right_fy42_Link, child rh6_right_fy43_Link, origin xyz=0.043692 -0.011217 0 rpy=1.5708 1.5704 1.5873, axis 0 0 -1, limit lower=0 upper=0 effort=0 velocity=0
- added joint rh6_right_fy51: type revolute, parent rh6_right_base_link, child rh6_right_fy51_Link, origin xyz=-0.0035 -0.029624 0.10795 rpy=3.1416 -1.4923 -1.5708, axis 0 0 -1, limit lower=0 upper=1.545 effort=0 velocity=0
- added joint rh6_right_fy52: type revolute, parent rh6_right_fy51_Link, child rh6_right_fy52_Link, origin xyz=0.0369 0.001 0 rpy=0 0 0, axis 0 0 -1, limit lower=0 upper=1.658 effort=0 velocity=0
- added joint rh6_right_fy53: type revolute, parent rh6_right_fy52_Link, child rh6_right_fy53_Link, origin xyz=0.043691 -0.011217 0 rpy=1.5708 1.5695 1.5873, axis 0 0 -1, limit lower=0 upper=0 effort=0 velocity=0
